File: Project_1_LED_Torch/Project_1_LED_Torch.kicad_pcb (KiCad board)
At the start: 2 copper layers, 4 parts, among them SW1 SW_DPDT_x2

Commit message: update v2
Parts:
- added REF**: MountingHole_2.1mm, MountingHole:MountingHole_2.1mm, F.Cu at (116.5, 63.0)
- moved D1 50.1 mm to (110.5, 61.7), turned to -90 degrees
- moved SW1 37.9 mm to (124.8, 60.8)
- moved R1 31.2 mm to (121.0, 66.8), turned to 90 degrees
- moved BT1 19.6 mm to (150.0, 63.0), turned to 180 degrees
Routing:
- net /bat_pos: track 0.00 -> 41.1 mm
- net /LED_cathode: track 0.00 -> 26.8 mm
- net /LED_anode: track 0.00 -> 11.6 mm
- net Net-(SW1A-A): track 0.00 -> 10.9 mm
Other:
- board outline added: 62 x 27.1 mm

Commit message: hehehe
Parts:
- added REF**: KiCad-Logo2_6mm_SilkScreen, Symbol:KiCad-Logo2_6mm_SilkScreen, B.Cu at (150.0, 62.5)
Other:
- board text added: "+"
- board text added: "-"
